Commit message: h

File: descriptions_pkg/descriptions/tebo_main.urdf.xacro (robot description, xacro)
@@ -1,6 +1,4 @@
 <?xml version="1.0"?>
 <robot xmlns:xacro="http://www.ros.org/wiki/xacro"  name="robot">
-    <xacro:include filename="robot_core.xacro" />
-    <xacro:include filename="gazebo_control.xacro" />
-    <xacro:include filename="lidar.xacro" />
+    <xacro:include filename="tebo_shape.xacro" />
 </robot>

File: descriptions_pkg/descriptions/tebo_params.xacro (robot description, xacro)
@@ -2,6 +2,18 @@
 <robot xmlns:xacro="http://ros.org/wiki/xacro">
   <!-- Define parameters -->
-  <xacro:property name="arm_length" value="1" />
-  <xacro:property name="arm_radius" value="0.1" />
+    <xacro:property name="chassis_length" value="0.335"/>
+    <xacro:property name="chassis_width" value="0.265"/>
+    <xacro:property name="chassis_height" value="0.138"/>
+    <xacro:property name="chassis_mass" value="1.0"/>
+    <xacro:property name="wheel_radius" value="0.033"/>
+    <xacro:property name="wheel_thickness" value="0.026"/>
+    <xacro:property name="wheel_mass" value="0.05"/>
+    <xacro:property name="wheel_offset_x" value="0.226"/>
+    <xacro:property name="wheel_offset_y" value="0.1485"/>
+    <xacro:property name="wheel_offset_z" value="0.01"/>
+    <xacro:property name="caster_wheel_radius" value="0.01"/>
+    <xacro:property name="caster_wheel_mass" value="0.01"/>
+    <xacro:property name="caster_wheel_offset_x" value="0.075"/>
+    <xacro:property name="caster_wheel_offset_z" value="${wheel_offset_z - wheel_radius + caster_wheel_radius}"/>
   <!-- ___INERTIAL-MACROS___ -->
     <xacro:macro name="inertial_sphere" params="mass radius *origin">

Commit message: h

File: descriptions_pkg/descriptions/tebo_main.urdf.xacro (robot description, xacro)
@@ -2,3 +2,5 @@
 <robot xmlns:xacro="http://www.ros.org/wiki/xacro"  name="robot">
     <xacro:include filename="tebo_shape.xacro" />
+    <xacro:include filename="tebo_gazebo.xacro"/>
+    <xacro:include filename="tebo_Glidar.xacro"/>
 </robot>

File: descriptions_pkg/descriptions/tebo_params.xacro (robot description, xacro)
@@ -12,6 +12,6 @@
     <xacro:property name="wheel_offset_y" value="0.1485"/>
     <xacro:property name="wheel_offset_z" value="0.01"/>
-    <xacro:property name="caster_wheel_radius" value="0.01"/>
-    <xacro:property name="caster_wheel_mass" value="0.01"/>
+    <xacro:property name="caster_wheel_radius" value="0.05"/>
+    <xacro:property name="caster_wheel_mass" value="0.1"/>
     <xacro:property name="caster_wheel_offset_x" value="0.075"/>
     <xacro:property name="caster_wheel_offset_z" value="${wheel_offset_z - wheel_radius + caster_wheel_radius}"/>

File: descriptions_pkg/descriptions/tebo_shape.xacro (robot description, xacro)
@@ -90,5 +90,5 @@
     </link>
     <gazebo reference="right_wheel">
-        <material>Gazebo/Orange</material>
+        <material>Gazebo/Blue</material>
     </gazebo>
     <!-- CASTER WHEEL LINK -->
