Commit message: h

File: descriptions_pkg/descriptions/tebo_Glidar.xacro (robot description, xacro)
@@ -23,5 +23,5 @@
     </link>
     <gazebo reference="laser_frame">
-        <material>Gazebo/Red</material>
+        <material>Gazebo/Black</material>
         <sensor name="laser" type="ray">
             <pose> 0 0 0 0 0 0 </pose>

File: descriptions_pkg/descriptions/tebo_main.urdf.xacro (robot description, xacro)
@@ -2,5 +2,5 @@
 <robot xmlns:xacro="http://www.ros.org/wiki/xacro"  name="robot">
     <xacro:include filename="tebo_shape.xacro" />
-    <xacro:include filename="tebo_gazebo.xacro"/>
+    <xacro:include filename="tebo_ros2_control.xacro"/>
     <xacro:include filename="tebo_Glidar.xacro"/>
 </robot>

File: descriptions_pkg/descriptions/tebo_params.xacro (robot description, xacro)
@@ -6,5 +6,5 @@
     <xacro:property name="chassis_height" value="0.138"/>
     <xacro:property name="chassis_mass" value="1.0"/>
-    <xacro:property name="wheel_radius" value="0.033"/>
+    <xacro:property name="wheel_radius" value="0.1"/>
     <xacro:property name="wheel_thickness" value="0.026"/>
     <xacro:property name="wheel_mass" value="0.05"/>

File: descriptions_pkg/descriptions/tebo_shape.xacro (robot description, xacro)
@@ -40,4 +40,22 @@
         <material>Gazebo/White</material>
     </gazebo>
+    <!-- ____LOGO____ -->
+    <joint name="face_joint" type="fixed">
+        <parent link="chassis"/>
+        <child link="text_link"/>
+        <origin xyz="${chassis_length} 0 ${chassis_height/2}" rpy="0 0 0"/>
+    </joint>
+    <link name="text_link">
+      <visual>
+        <origin xyz="0.01 0.005 0.01" rpy="${pi/2} 0 ${pi/2}"/>
+         <geometry>
+          <mesh filename="/home/danana/Downloads/ImageToStl.com_dark.stl" scale="0.002 0.002 0.002" />
+        </geometry>
+        <material name="blue"/>
+      </visual>
+    </link>
+    <gazebo reference="text_link">
+        <material>Gazebo/Blue</material>
+    </gazebo>
     <!-- LEFT WHEEL LINK -->
     <joint name="left_wheel_joint" type="continuous">
@@ -52,5 +70,5 @@
                 <cylinder radius="${wheel_radius}" length="${wheel_thickness}"/>
             </geometry>
-            <material name="blue"/>
+            <material name="orange"/>
         </visual>
         <collision>
@@ -64,5 +82,5 @@
     </link>
     <gazebo reference="left_wheel">
-        <material>Gazebo/Blue</material>
+        <material>Gazebo/Orange</material>
     </gazebo>
     <!-- RIGHT WHEEL LINK -->
@@ -78,5 +96,5 @@
                 <cylinder radius="${wheel_radius}" length="${wheel_thickness}"/>
             </geometry>
-            <material name="blue"/>
+            <material name="orange"/>
         </visual>
         <collision>
@@ -90,5 +108,5 @@
     </link>
     <gazebo reference="right_wheel">
-        <material>Gazebo/Blue</material>
+        <material>Gazebo/Orange</material>
     </gazebo>
     <!-- CASTER WHEEL LINK -->
@@ -103,5 +121,5 @@
                 <sphere radius="${caster_wheel_radius}"/>
             </geometry>
-            <material name="white"/>
+            <material name="black"/>
         </visual>
         <collision>
@@ -115,5 +133,5 @@
     </link>
     <gazebo reference="caster_wheel">
-        <material>Gazebo/Orange</material>
+        <material>Gazebo/Black</material>
         <mu1 value="0.001"/>
         <mu2 value="0.001"/>
